File: hardware/vancouver-skytrain-pcb/vancouver-skytrain-pcb.kicad_pcb (KiCad board)
At the start: 2 copper layers, 157 parts, among them J2_POWER_IN1 Conn_01x02, J3_PROGRAMING_PIN1 Conn_01x06, Q1 PN2222A, Q2 PN2222A, U1 74AHC1G125, U2 74AHC1G125, U3 74AHC1G125, U4 74AHC1G125

Commit message: positioned all the LEDs, Cap, and 5v Rails
Parts:
- removed the G*** at (180.5, 122.0)
- removed U2, U3, U4: 74AHC1G125, Package_TO_SOT_SMD:SOT-23-5
- added C100: 1uF,25V,X5R, vancouver-skytrain-pcb.pretty:C_0402_1005Metric, F.Cu at (207.0, 103.9)
- added C101: 1uF,25V,X5R, vancouver-skytrain-pcb.pretty:C_0402_1005Metric, F.Cu at (207.0, 106.9)
- added C102: 1uF,25V,X5R, vancouver-skytrain-pcb.pretty:C_0402_1005Metric, F.Cu at (197.2, 103.8)
- added C103: 10uF,10V,X5R, vancouver-skytrain-pcb.pretty:C_0603_1608Metric, F.Cu at (348.0, 143.0)
- added C104: 1uF,25V,X5R, vancouver-skytrain-pcb.pretty:C_0402_1005Metric, F.Cu at (197.2, 107.0)
- added C105: 1uF,25V,X5R, vancouver-skytrain-pcb.pretty:C_0402_1005Metric, F.Cu at (285.2, 73.5)
- added C106: 1uF,25V,X5R, vancouver-skytrain-pcb.pretty:C_0402_1005Metric, F.Cu at (266.8, 107.5)
- added C107: 1uF,25V,X5R, vancouver-skytrain-pcb.pretty:C_0402_1005Metric, F.Cu at (261.8, 107.5)
- added C108: 1uF,25V,X5R, vancouver-skytrain-pcb.pretty:C_0402_1005Metric, F.Cu at (261.8, 104.0)
- added C109: 1uF,25V,X5R, vancouver-skytrain-pcb.pretty:C_0402_1005Metric, F.Cu at (266.8, 104.0)
- added C110: 1uF,25V,X5R, vancouver-skytrain-pcb.pretty:C_0402_1005Metric, F.Cu at (257.0, 107.3)
- added C111: 1uF,25V,X5R, vancouver-skytrain-pcb.pretty:C_0402_1005Metric, F.Cu at (257.0, 104.0)
- added C112: 1uF,25V,X5R, vancouver-skytrain-pcb.pretty:C_0402_1005Metric, F.Cu at (252.2, 104.0)
- added C113: 1uF,25V,X5R, vancouver-skytrain-pcb.pretty:C_0402_1005Metric, F.Cu at (252.2, 107.3)
- added C114: 1uF,25V,X5R, vancouver-skytrain-pcb.pretty:C_0402_1005Metric, F.Cu at (244.2, 104.0)
- added C115: 1uF,25V,X5R, vancouver-skytrain-pcb.pretty:C_0402_1005Metric, F.Cu at (244.2, 107.2)
- added C116: 1uF,25V,X5R, vancouver-skytrain-pcb.pretty:C_0402_1005Metric, F.Cu at (231.8, 104.0)
- added C117: 1uF,25V,X5R, vancouver-skytrain-pcb.pretty:C_0402_1005Metric, F.Cu at (231.8, 107.2)
- added C118: 1uF,25V,X5R, vancouver-skytrain-pcb.pretty:C_0402_1005Metric, F.Cu at (219.2, 103.9)
- added C119: 1uF,25V,X5R, vancouver-skytrain-pcb.pretty:C_0402_1005Metric, F.Cu at (275.0, 84.8)
- added C120: 10uF,10V,X5R, vancouver-skytrain-pcb.pretty:C_0603_1608Metric, F.Cu at (348.0, 145.5)
- added C121: 1uF,25V,X5R, vancouver-skytrain-pcb.pretty:C_0402_1005Metric, F.Cu at (271.8, 84.8)
- added C122: 1uF,25V,X5R, vancouver-skytrain-pcb.pretty:C_0402_1005Metric, F.Cu at (269.8, 118.0)
- added C123: 1uF,25V,X5R, vancouver-skytrain-pcb.pretty:C_0402_1005Metric, F.Cu at (365.0, 138.2)
- added C124: 1uF,25V,X5R, vancouver-skytrain-pcb.pretty:C_0402_1005Metric, F.Cu at (285.2, 77.0)
- added C125: 1uF,25V,X5R, vancouver-skytrain-pcb.pretty:C_0402_1005Metric, F.Cu at (296.8, 73.5)
- added C126: 1uF,25V,X5R, vancouver-skytrain-pcb.pretty:C_0402_1005Metric, F.Cu at (296.8, 77.0)
- added C127: 1uF,25V,X5R, vancouver-skytrain-pcb.pretty:C_0402_1005Metric, F.Cu at (311.5, 76.8)
- added C128: 1uF,25V,X5R, vancouver-skytrain-pcb.pretty:C_0402_1005Metric, F.Cu at (308.8, 74.2)
- added C129: 1uF,25V,X5R, vancouver-skytrain-pcb.pretty:C_0402_1005Metric, F.Cu at (310.0, 67.0)
- added C130: 1uF,25V,X5R, vancouver-skytrain-pcb.pretty:C_0402_1005Metric, F.Cu at (313.5, 67.0)
- added C131: 1uF,25V,X5R, vancouver-skytrain-pcb.pretty:C_0402_1005Metric, F.Cu at (310.0, 58.0)
- added C132: 1uF,25V,X5R, vancouver-skytrain-pcb.pretty:C_0402_1005Metric, F.Cu at (313.5, 58.0)
- added C133: 1uF,25V,X5R, vancouver-skytrain-pcb.pretty:C_0402_1005Metric, F.Cu at (267.2, 115.5)
- added C134: 1uF,25V,X5R, vancouver-skytrain-pcb.pretty:C_0402_1005Metric, F.Cu at (271.5, 157.2)
- added C135: 1uF,25V,X5R, vancouver-skytrain-pcb.pretty:C_0402_1005Metric, F.Cu at (275.2, 157.2)
- added C136: 1uF,25V,X5R, vancouver-skytrain-pcb.pretty:C_0402_1005Metric, F.Cu at (271.5, 168.2)
- added C137: 10uF,10V,X5R, vancouver-skytrain-pcb.pretty:C_0603_1608Metric, F.Cu at (348.0, 148.0)
- added C138: 1uF,25V,X5R, vancouver-skytrain-pcb.pretty:C_0402_1005Metric, F.Cu at (275.2, 168.2)
- added C139: 1uF,25V,X5R, vancouver-skytrain-pcb.pretty:C_0402_1005Metric, F.Cu at (362.7, 133.1)
- added C140: 10uF,10V,X5R, vancouver-skytrain-pcb.pretty:C_0603_1608Metric, F.Cu at (348.0, 150.5)
- added C141: 1uF,25V,X5R, vancouver-skytrain-pcb.pretty:C_0402_1005Metric, F.Cu at (362.7, 135.1)
- added C142: 1uF,25V,X5R, vancouver-skytrain-pcb.pretty:C_0402_1005Metric, F.Cu at (366.0, 134.8)
- added C74: 1uF,25V,X5R, vancouver-skytrain-pcb.pretty:C_0402_1005Metric, F.Cu at (183.8, 107.0)
- added C75: 1uF,25V,X5R, vancouver-skytrain-pcb.pretty:C_0402_1005Metric, F.Cu at (112.0, 107.0)
- added C76: 1uF,25V,X5R, vancouver-skytrain-pcb.pretty:C_0402_1005Metric, F.Cu at (113.8, 116.2)
- added C77: 1uF,25V,X5R, vancouver-skytrain-pcb.pretty:C_0402_1005Metric, F.Cu at (117.0, 116.2)
- added C78: 1uF,25V,X5R, vancouver-skytrain-pcb.pretty:C_0402_1005Metric, F.Cu at (113.7, 129.0)
- added C79: 10uF,10V,X5R, vancouver-skytrain-pcb.pretty:C_0603_1608Metric, F.Cu at (348.0, 140.5)
- added C80: 1uF,25V,X5R, vancouver-skytrain-pcb.pretty:C_0402_1005Metric, F.Cu at (117.0, 129.0)
- added C81: 1uF,25V,X5R, vancouver-skytrain-pcb.pretty:C_0402_1005Metric, F.Cu at (113.8, 144.0)
- added C82: 1uF,25V,X5R, vancouver-skytrain-pcb.pretty:C_0402_1005Metric, F.Cu at (117.0, 144.0)
- added C83: 1uF,25V,X5R, vancouver-skytrain-pcb.pretty:C_0402_1005Metric, F.Cu at (117.0, 154.0)
- added C84: 1uF,25V,X5R, vancouver-skytrain-pcb.pretty:C_0402_1005Metric, F.Cu at (113.8, 154.2)
- added C85: 1uF,25V,X5R, vancouver-skytrain-pcb.pretty:C_0402_1005Metric, F.Cu at (113.8, 166.2)
- added C86: 1uF,25V,X5R, vancouver-skytrain-pcb.pretty:C_0402_1005Metric, F.Cu at (117.0, 166.2)
- added C87: 1uF,25V,X5R, vancouver-skytrain-pcb.pretty:C_0402_1005Metric, F.Cu at (113.7, 176.5)
- added C88: 1uF,25V,X5R, vancouver-skytrain-pcb.pretty:C_0402_1005Metric, F.Cu at (117.0, 176.5)
- added C89: 1uF,25V,X5R, vancouver-skytrain-pcb.pretty:C_0402_1005Metric, F.Cu at (117.0, 186.5)
- added C90: 1uF,25V,X5R, vancouver-skytrain-pcb.pretty:C_0402_1005Metric, F.Cu at (113.8, 186.5)
- added C91: 1uF,25V,X5R, vancouver-skytrain-pcb.pretty:C_0402_1005Metric, F.Cu at (113.8, 196.8)
- added C92: 1uF,25V,X5R, vancouver-skytrain-pcb.pretty:C_0402_1005Metric, F.Cu at (117.0, 196.8)
- added C93: 1uF,25V,X5R, vancouver-skytrain-pcb.pretty:C_0402_1005Metric, F.Cu at (97.2, 174.8)
- added C94: 1uF,25V,X5R, vancouver-skytrain-pcb.pretty:C_0402_1005Metric, F.Cu at (97.2, 171.5)
- added C95: 1uF,25V,X5R, vancouver-skytrain-pcb.pretty:C_0402_1005Metric, F.Cu at (87.2, 174.8)
- added C96: 1uF,25V,X5R, vancouver-skytrain-pcb.pretty:C_0402_1005Metric, F.Cu at (87.2, 171.5)
- added C97: 1uF,25V,X5R, vancouver-skytrain-pcb.pretty:C_0402_1005Metric, F.Cu at (77.0, 174.8)
- added C98: 1uF,25V,X5R, vancouver-skytrain-pcb.pretty:C_0402_1005Metric, F.Cu at (77.0, 171.5)
- added C99: 1uF,25V,X5R, vancouver-skytrain-pcb.pretty:C_0402_1005Metric, F.Cu at (219.2, 107.2)
- added G*** (x3): LOGO, LOGO, F.Cu at (175.5, 124.9)
- added LED100: WS2812B, vancouver-skytrain-pcb.pretty:XL-1010RGBC-WS2812B, F.Cu at (116.2, 145.7)
- added LED101: WS2812B, vancouver-skytrain-pcb.pretty:XL-1010RGBC-WS2812B, F.Cu at (116.3, 130.5)
- added LED102: WS2812B, vancouver-skytrain-pcb.pretty:XL-1010RGBC-WS2812B, F.Cu at (116.3, 117.9)
- added LED103: WS2812B, vancouver-skytrain-pcb.pretty:XL-1010RGBC-WS2812B, F.Cu at (113.7, 104.4)
- added LED104: WS2812B, vancouver-skytrain-pcb.pretty:XL-1010RGBC-WS2812B, F.Cu at (116.4, 98.0)
- added LED105: WS2812B, vancouver-skytrain-pcb.pretty:XL-1010RGBC-WS2812B, F.Cu at (105.6, 85.2)
- added LED106: WS2812B, vancouver-skytrain-pcb.pretty:XL-1010RGBC-WS2812B, F.Cu at (100.6, 73.4)
- added LED107: WS2812B, vancouver-skytrain-pcb.pretty:XL-1010RGBC-WS2812B, F.Cu at (112.0, 61.4)
- added LED108: WS2812B, vancouver-skytrain-pcb.pretty:XL-1010RGBC-WS2812B, F.Cu at (110.7, 60.1)
- added LED109: WS2812B, vancouver-skytrain-pcb.pretty:XL-1010RGBC-WS2812B, F.Cu at (99.3, 72.1)
- added LED110: WS2812B, vancouver-skytrain-pcb.pretty:XL-1010RGBC-WS2812B, F.Cu at (104.3, 86.4)
- added LED111: WS2812B, vancouver-skytrain-pcb.pretty:XL-1010RGBC-WS2812B, F.Cu at (114.6, 98.0)
- added LED112: WS2812B, vancouver-skytrain-pcb.pretty:XL-1010RGBC-WS2812B, F.Cu at (113.7, 106.2)
- added LED113: WS2812B, vancouver-skytrain-pcb.pretty:XL-1010RGBC-WS2812B, F.Cu at (114.5, 117.9)
- added LED114: WS2812B, vancouver-skytrain-pcb.pretty:XL-1010RGBC-WS2812B, F.Cu at (114.6, 130.5)
- added LED115: WS2812B, vancouver-skytrain-pcb.pretty:XL-1010RGBC-WS2812B, F.Cu at (114.4, 145.7)
- added LED116: WS2812B, vancouver-skytrain-pcb.pretty:XL-1010RGBC-WS2812B, F.Cu at (114.5, 155.4)
- added LED117: WS2812B, vancouver-skytrain-pcb.pretty:XL-1010RGBC-WS2812B, F.Cu at (114.5, 167.8)
- added LED118: WS2812B, vancouver-skytrain-pcb.pretty:XL-1010RGBC-WS2812B, F.Cu at (95.6, 172.3)
- added LED119: WS2812B, vancouver-skytrain-pcb.pretty:XL-1010RGBC-WS2812B, F.Cu at (85.6, 172.3)
- added LED120: WS2812B, vancouver-skytrain-pcb.pretty:XL-1010RGBC-WS2812B, F.Cu at (75.6, 172.3)
- added LED121: WS2812B, vancouver-skytrain-pcb.pretty:XL-1010RGBC-WS2812B, F.Cu at (75.6, 174.2)
- added LED122: WS2812B, vancouver-skytrain-pcb.pretty:XL-1010RGBC-WS2812B, F.Cu at (85.7, 174.0)
- added LED123: WS2812B, vancouver-skytrain-pcb.pretty:XL-1010RGBC-WS2812B, F.Cu at (95.6, 174.1)
- added LED124: WS2812B, vancouver-skytrain-pcb.pretty:XL-1010RGBC-WS2812B, F.Cu at (114.5, 178.1)
- added LED125: WS2812B, vancouver-skytrain-pcb.pretty:XL-1010RGBC-WS2812B, F.Cu at (114.6, 188.2)
- added LED126: WS2812B, vancouver-skytrain-pcb.pretty:XL-1010RGBC-WS2812B, F.Cu at (114.7, 198.2)
- added LED66: WS2812B, vancouver-skytrain-pcb.pretty:XL-1010RGBC-WS2812B, F.Cu at (133.0, 97.2)
- added LED67: WS2812B, vancouver-skytrain-pcb.pretty:XL-1010RGBC-WS2812B, F.Cu at (125.2, 104.7)
- added LED68: WS2812B, vancouver-skytrain-pcb.pretty:XL-1010RGBC-WS2812B, F.Cu at (115.5, 104.5)
- added LED69: WS2812B, vancouver-skytrain-pcb.pretty:XL-1010RGBC-WS2812B, F.Cu at (105.5, 104.6)
- added LED70: WS2812B, vancouver-skytrain-pcb.pretty:XL-1010RGBC-WS2812B, F.Cu at (95.5, 104.7)
- added LED71: WS2812B, vancouver-skytrain-pcb.pretty:XL-1010RGBC-WS2812B, F.Cu at (85.9, 104.6)
- added LED72: WS2812B, vancouver-skytrain-pcb.pretty:XL-1010RGBC-WS2812B, F.Cu at (85.9, 106.4)
- added LED73: WS2812B, vancouver-skytrain-pcb.pretty:XL-1010RGBC-WS2812B, F.Cu at (95.5, 106.4)
- added LED74: WS2812B, vancouver-skytrain-pcb.pretty:XL-1010RGBC-WS2812B, F.Cu at (105.5, 106.4)
- added LED75: WS2812B, vancouver-skytrain-pcb.pretty:XL-1010RGBC-WS2812B, F.Cu at (115.5, 106.2)
- added LED76: WS2812B, vancouver-skytrain-pcb.pretty:XL-1010RGBC-WS2812B, F.Cu at (125.2, 106.5)
- added LED77: WS2812B, vancouver-skytrain-pcb.pretty:XL-1010RGBC-WS2812B, F.Cu at (133.0, 98.9)
- added LED78: WS2812B, vancouver-skytrain-pcb.pretty:XL-1010RGBC-WS2812B, F.Cu at (144.7, 98.8)
- added LED79: WS2812B, vancouver-skytrain-pcb.pretty:XL-1010RGBC-WS2812B, F.Cu at (153.8, 105.3)
- added LED80: WS2812B, vancouver-skytrain-pcb.pretty:XL-1010RGBC-WS2812B, F.Cu at (168.9, 106.3)
- added LED81: WS2812B, vancouver-skytrain-pcb.pretty:XL-1010RGBC-WS2812B, F.Cu at (182.1, 106.3)
- added LED82: WS2812B, vancouver-skytrain-pcb.pretty:XL-1010RGBC-WS2812B, F.Cu at (195.4, 106.4)
- added LED83: WS2812B, vancouver-skytrain-pcb.pretty:XL-1010RGBC-WS2812B, F.Cu at (205.3, 106.3)
- added LED84: WS2812B, vancouver-skytrain-pcb.pretty:XL-1010RGBC-WS2812B, F.Cu at (217.6, 106.4)
- added LED85: WS2812B, vancouver-skytrain-pcb.pretty:XL-1010RGBC-WS2812B, F.Cu at (230.0, 106.4)
- added LED86: WS2812B, vancouver-skytrain-pcb.pretty:XL-1010RGBC-WS2812B, F.Cu at (242.4, 106.4)
- added LED87: WS2812B, vancouver-skytrain-pcb.pretty:XL-1010RGBC-WS2812B, F.Cu at (253.8, 106.4)
- added LED88: WS2812B, vancouver-skytrain-pcb.pretty:XL-1010RGBC-WS2812B, F.Cu at (263.3, 106.6)
- added LED89: WS2812B, vancouver-skytrain-pcb.pretty:XL-1010RGBC-WS2812B, F.Cu at (274.2, 83.2)
- added LED90: WS2812B, vancouver-skytrain-pcb.pretty:XL-1010RGBC-WS2812B, F.Cu at (286.9, 76.1)
- added LED91: WS2812B, vancouver-skytrain-pcb.pretty:XL-1010RGBC-WS2812B, F.Cu at (298.3, 76.1)
- added LED92: WS2812B, vancouver-skytrain-pcb.pretty:XL-1010RGBC-WS2812B, F.Cu at (312.0, 75.0)
- added LED93: WS2812B, vancouver-skytrain-pcb.pretty:XL-1010RGBC-WS2812B, F.Cu at (312.8, 65.4)
- added LED94: WS2812B, vancouver-skytrain-pcb.pretty:XL-1010RGBC-WS2812B, F.Cu at (312.8, 56.6)
- added LED95: WS2812B, vancouver-skytrain-pcb.pretty:XL-1010RGBC-WS2812B, F.Cu at (116.5, 198.3)
- added LED96: WS2812B, vancouver-skytrain-pcb.pretty:XL-1010RGBC-WS2812B, F.Cu at (116.3, 188.2)
- added LED97: WS2812B, vancouver-skytrain-pcb.pretty:XL-1010RGBC-WS2812B, F.Cu at (116.2, 178.1)
- added LED98: WS2812B, vancouver-skytrain-pcb.pretty:XL-1010RGBC-WS2812B, F.Cu at (116.2, 167.8)
- added LED99: WS2812B, vancouver-skytrain-pcb.pretty:XL-1010RGBC-WS2812B, F.Cu at (116.3, 155.5)
- C54, C71: value 10uF,10V,X5R -> 1uF,25V,X5R; footprint vancouver-skytrain-pcb.pretty:C_0603_1608Metric -> vancouver-skytrain-pcb.pretty:C_0402_1005Metric
- C55: value 1uF,25V,X5R -> 10uF,10V,X5R; footprint vancouver-skytrain-pcb.pretty:C_0402_1005Metric -> vancouver-skytrain-pcb.pretty:C_0603_1608Metric
- LED1, LED10, LED11, LED12, LED13, LED14, LED15, LED16, LED17, LED18, LED19, LED2, LED20, LED21, LED22, LED23, LED24, LED25, LED26, LED27, LED28, LED29, LED3, LED30, LED31, LED32, LED33, LED34, LED35, LED36, LED37, LED38, LED39, LED4, LED40, LED41, LED42, LED43, LED44, LED45, LED46, LED47, LED48, LED49, LED5, LED50, LED51, LED52, LED53, LED54, LED55, LED56, LED57, LED58, LED59, LED6, LED60, LED61, LED62, LED63, LED64, LED65, LED7, LED8, LED9: footprint LED_SMD:LED_WS2812B_PLCC4_5.0x5.0mm_P3.2mm -> vancouver-skytrain-pcb.pretty:XL-1010RGBC-WS2812B
- moved C40 395.8 mm to (87.5, 107.2), turned to 90 degrees
- moved C41 394.3 mm to (87.5, 103.8), turned to -90 degrees
- moved C43 385.0 mm to (97.0, 107.2), turned to 90 degrees
- moved C42 384.6 mm to (97.0, 103.8), turned to -90 degrees
- moved C45 374.3 mm to (107.0, 107.2), turned to 90 degrees
- moved C44 373.9 mm to (107.0, 103.8), turned to -90 degrees
- moved C66 373.7 mm to (105.0, 62.5), turned to 135 degrees
- moved C67 373.4 mm to (107.2, 75.0), turned to 45 degrees
- moved C39 370.9 mm to (97.5, 72.8), turned to -45 degrees
- moved C34 370.5 mm to (100.0, 75.2), turned to 135 degrees
- moved C61 369.7 mm to (112.0, 103.5), turned to -90 degrees
- moved C37 367.0 mm to (105.0, 88.2), turned to 45 degrees
- moved C68 366.5 mm to (115.8, 83.2), turned to 45 degrees
- moved C62 365.3 mm to (117.0, 107.0), turned to 90 degrees
- moved C63 363.9 mm to (117.0, 103.5), turned to -90 degrees
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Connections:
- net LEDS_EXPO_LINE renamed LED_IN
- net Net-(LED1-DIN) renamed LEDS_EXPO_LINE_EAST_TO_WEST
- C54 pad 1: GND -> +5V
- C54 pad 2: +5V -> GND
- C55 pad 1: +5V -> GND
- C55 pad 2: GND -> +5V
- C71 pad 1: GND -> +5V
- C71 pad 2: +5V -> GND
- LED1 pad 1: +5V -> Net-(LED1-DOUT)
- LED1 pad 2: Net-(LED1-DOU) -> +5V
- LED10 pad 1: +5V -> Net-(LED10-DOUT)
- LED10 pad 2: Net-(LED10-DOU) -> +5V
- LED11 pad 1: +5V -> Net-(LED11-DOUT)
- LED11 pad 2: Net-(LED11-DOU) -> +5V
- LED11 pad 4: Net-(LED10-DOU) -> Net-(LED10-DOUT)
- LED12 pad 1: +5V -> Net-(LED12-DOUT)
- LED12 pad 2: Net-(LED12-DOU) -> +5V
- LED12 pad 4: Net-(LED11-DOU) -> Net-(LED11-DOUT)
- LED13 pad 1: +5V -> Net-(LED13-DOUT)
- LED13 pad 2: Net-(LED13-DOU) -> +5V
- LED13 pad 4: Net-(LED12-DOU) -> Net-(LED12-DOUT)
- LED14 pad 1: +5V -> Net-(LED14-DOUT)
- LED14 pad 2: Net-(LED14-DOU) -> +5V
- LED14 pad 4: Net-(LED13-DOU) -> Net-(LED13-DOUT)
- LED15 pad 1: +5V -> Net-(LED15-DOUT)
- LED15 pad 2: Net-(LED15-DOU) -> +5V
- LED15 pad 4: Net-(LED14-DOU) -> Net-(LED14-DOUT)
- LED16 pad 1: +5V -> Net-(LED16-DOUT)
- LED16 pad 2: Net-(LED16-DOU) -> +5V
- LED16 pad 4: Net-(LED15-DOU) -> Net-(LED15-DOUT)
- LED17 pad 1: +5V -> Net-(LED17-DOUT)
- LED17 pad 2: Net-(LED17-DOU) -> +5V
- LED17 pad 4: Net-(LED16-DOU) -> Net-(LED16-DOUT)
- LED18 pad 1: +5V -> Net-(LED18-DOUT)
- LED18 pad 2: Net-(LED18-DOU) -> +5V
- LED18 pad 4: Net-(LED17-DOU) -> Net-(LED17-DOUT)
- LED19 pad 1: +5V -> Net-(LED19-DOUT)
- LED19 pad 2: Net-(LED19-DOU) -> +5V
- LED19 pad 4: Net-(LED18-DOU) -> Net-(LED18-DOUT)
- LED2 pad 1: +5V -> Net-(LED2-DOUT)
- LED2 pad 2: Net-(LED2-DOU) -> +5V
- LED2 pad 4: Net-(LED1-DOU) -> Net-(LED1-DOUT)
- LED20 pad 1: +5V -> Net-(LED20-DOUT)
- LED20 pad 2: Net-(LED20-DOU) -> +5V
- LED20 pad 4: Net-(LED19-DOU) -> Net-(LED19-DOUT)
- LED21 pad 1: +5V -> Net-(LED21-DOUT)
- LED21 pad 2: Net-(LED21-DOU) -> +5V
- LED21 pad 4: Net-(LED20-DOU) -> Net-(LED20-DOUT)
- LED22 pad 1: +5V -> Net-(LED22-DOUT)
- LED22 pad 2: Net-(LED22-DOU) -> +5V
- LED22 pad 4: Net-(LED21-DOU) -> Net-(LED21-DOUT)
- LED23 pad 1: +5V -> Net-(LED23-DOUT)
- LED23 pad 2: Net-(LED23-DOU) -> +5V
- LED23 pad 4: Net-(LED22-DOU) -> Net-(LED22-DOUT)
- LED24 pad 1: +5V -> LEDS_EXPO_LINE_WEST_TO_EAST
- LED24 pad 2: unconnected-(LED24-DOU-Pad2) -> +5V
- LED24 pad 4: Net-(LED23-DOU) -> Net-(LED23-DOUT)
- LED25 pad 1: +5V -> Net-(LED25-DOUT)
- LED25 pad 2: Net-(LED25-DOU) -> +5V
- LED25 pad 4: Net-(LED25-DIN) -> LEDS_EXPO_LINE_WEST_TO_EAST
- LED26 pad 1: +5V -> Net-(LED26-DOUT)
- LED26 pad 2: Net-(LED26-DOU) -> +5V
- LED26 pad 4: Net-(LED25-DOU) -> Net-(LED25-DOUT)
- LED27 pad 1: +5V -> Net-(LED27-DOUT)
- LED27 pad 2: Net-(LED27-DOU) -> +5V
- LED27 pad 4: Net-(LED26-DOU) -> Net-(LED26-DOUT)
- LED28 pad 1: +5V -> Net-(LED28-DOUT)
- LED28 pad 2: Net-(LED28-DOU) -> +5V
- LED28 pad 4: Net-(LED27-DOU) -> Net-(LED27-DOUT)
- LED29 pad 1: +5V -> Net-(LED29-DOUT)
- LED29 pad 2: Net-(LED29-DOU) -> +5V
- LED29 pad 4: Net-(LED28-DOU) -> Net-(LED28-DOUT)
- LED3 pad 1: +5V -> Net-(LED3-DOUT)
- LED3 pad 2: Net-(LED3-DOU) -> +5V
- LED3 pad 4: Net-(LED2-DOU) -> Net-(LED2-DOUT)
- LED30 pad 1: +5V -> Net-(LED30-DOUT)
- LED30 pad 2: Net-(LED30-DOU) -> +5V
- LED30 pad 4: Net-(LED29-DOU) -> Net-(LED29-DOUT)
- LED31 pad 1: +5V -> Net-(LED31-DOUT)
- LED31 pad 2: Net-(LED31-DOU) -> +5V
- LED31 pad 4: Net-(LED30-DOU) -> Net-(LED30-DOUT)
- LED32 pad 1: +5V -> Net-(LED32-DOUT)
- LED32 pad 2: Net-(LED32-DOU) -> +5V
- LED32 pad 4: Net-(LED31-DOU) -> Net-(LED31-DOUT)
- LED33 pad 1: +5V -> Net-(LED33-DOUT)
- LED33 pad 2: Net-(LED33-DOU) -> +5V
- LED33 pad 4: Net-(LED32-DOU) -> Net-(LED32-DOUT)
- LED34 pad 1: +5V -> Net-(LED34-DOUT)
- LED34 pad 2: Net-(LED34-DOU) -> +5V
- LED34 pad 4: Net-(LED33-DOU) -> Net-(LED33-DOUT)
- LED35 pad 1: +5V -> Net-(LED35-DOUT)
- LED35 pad 2: Net-(LED35-DOU) -> +5V
- LED35 pad 4: Net-(LED34-DOU) -> Net-(LED34-DOUT)
- LED36 pad 1: +5V -> Net-(LED36-DOUT)
- LED36 pad 2: Net-(LED36-DOU) -> +5V
- LED36 pad 4: Net-(LED35-DOU) -> Net-(LED35-DOUT)
- LED37 pad 1: +5V -> Net-(LED37-DOUT)
- LED37 pad 2: Net-(LED37-DOU) -> +5V
- LED37 pad 4: Net-(LED36-DOU) -> Net-(LED36-DOUT)
- LED38 pad 1: +5V -> Net-(LED38-DOUT)
- LED38 pad 2: Net-(LED38-DOU) -> +5V
- LED38 pad 4: Net-(LED37-DOU) -> Net-(LED37-DOUT)
- LED39 pad 1: +5V -> Net-(LED39-DOUT)
- LED39 pad 2: Net-(LED39-DOU) -> +5V
- LED39 pad 4: Net-(LED38-DOU) -> Net-(LED38-DOUT)
- LED4 pad 1: +5V -> Net-(LED4-DOUT)
- LED4 pad 2: Net-(LED4-DOU) -> +5V
- LED4 pad 4: Net-(LED3-DOU) -> Net-(LED3-DOUT)
- LED40 pad 1: +5V -> Net-(LED40-DOUT)
- LED40 pad 2: Net-(LED40-DOU) -> +5V
- LED40 pad 4: Net-(LED39-DOU) -> Net-(LED39-DOUT)
- LED41 pad 1: +5V -> Net-(LED41-DOUT)
- LED41 pad 2: Net-(LED41-DOU) -> +5V
- LED41 pad 4: Net-(LED40-DOU) -> Net-(LED40-DOUT)
- LED42 pad 1: +5V -> Net-(LED42-DOUT)
- LED42 pad 2: Net-(LED42-DOU) -> +5V
- LED42 pad 4: Net-(LED41-DOU) -> Net-(LED41-DOUT)
- LED43 pad 1: +5V -> Net-(LED43-DOUT)
- LED43 pad 2: Net-(LED43-DOU) -> +5V
- LED43 pad 4: Net-(LED42-DOU) -> Net-(LED42-DOUT)
- LED44 pad 1: +5V -> Net-(LED44-DOUT)
- LED44 pad 2: Net-(LED44-DOU) -> +5V
- LED44 pad 4: Net-(LED43-DOU) -> Net-(LED43-DOUT)
- LED45 pad 1: +5V -> Net-(LED45-DOUT)
- LED45 pad 2: Net-(LED45-DOU) -> +5V
- LED45 pad 4: Net-(LED44-DOU) -> Net-(LED44-DOUT)
- LED46 pad 1: +5V -> Net-(LED46-DOUT)
- LED46 pad 2: Net-(LED46-DOU) -> +5V
- LED46 pad 4: Net-(LED45-DOU) -> Net-(LED45-DOUT)
- LED47 pad 1: +5V -> Net-(LED47-DOUT)
- LED47 pad 2: unconnected-(LED47-DOU-Pad2) -> +5V
- LED47 pad 4: Net-(LED46-DOU) -> Net-(LED46-DOUT)
- LED48 pad 1: +5V -> LEDS_MILLENNIUM_LINE_EAST_TO_WEST
- LED48 pad 2: Net-(LED48-DOU) -> +5V
- LED48 pad 4: Net-(LED48-DIN) -> Net-(LED47-DOUT)
- LED49 pad 1: +5V -> Net-(LED49-DOUT)
- LED49 pad 2: Net-(LED49-DOU) -> +5V
- LED49 pad 4: Net-(LED48-DOU) -> LEDS_MILLENNIUM_LINE_EAST_TO_WEST
- LED5 pad 1: +5V -> Net-(LED5-DOUT)
- LED5 pad 2: Net-(LED5-DOU) -> +5V
- LED5 pad 4: Net-(LED4-DOU) -> Net-(LED4-DOUT)
- LED50 pad 1: +5V -> Net-(LED50-DOUT)
- LED50 pad 2: Net-(LED50-DOU) -> +5V
- LED50 pad 4: Net-(LED49-DOU) -> Net-(LED49-DOUT)
- LED51 pad 1: +5V -> Net-(LED51-DOUT)
- LED51 pad 2: Net-(LED51-DOU) -> +5V
- LED51 pad 4: Net-(LED50-DOU) -> Net-(LED50-DOUT)
- LED52 pad 1: +5V -> Net-(LED52-DOUT)
- LED52 pad 2: Net-(LED52-DOU) -> +5V
- LED52 pad 4: Net-(LED51-DOU) -> Net-(LED51-DOUT)
- LED53 pad 1: +5V -> Net-(LED53-DOUT)
- LED53 pad 2: Net-(LED53-DOU) -> +5V
- LED53 pad 4: Net-(LED52-DOU) -> Net-(LED52-DOUT)
- LED54 pad 1: +5V -> Net-(LED54-DOUT)
- LED54 pad 2: Net-(LED54-DOU) -> +5V
- LED54 pad 4: Net-(LED53-DOU) -> Net-(LED53-DOUT)
- LED55 pad 1: +5V -> Net-(LED55-DOUT)
- LED55 pad 2: Net-(LED55-DOU) -> +5V
- LED55 pad 4: Net-(LED54-DOU) -> Net-(LED54-DOUT)
- LED56 pad 1: +5V -> Net-(LED56-DOUT)
- LED56 pad 2: Net-(LED56-DOU) -> +5V
- LED56 pad 4: Net-(LED55-DOU) -> Net-(LED55-DOUT)
- LED57 pad 1: +5V -> Net-(LED57-DOUT)
- LED57 pad 2: Net-(LED57-DOU) -> +5V
- LED57 pad 4: Net-(LED56-DOU) -> Net-(LED56-DOUT)
- LED58 pad 1: +5V -> Net-(LED58-DOUT)
- LED58 pad 2: Net-(LED58-DOU) -> +5V
- LED58 pad 4: Net-(LED57-DOU) -> Net-(LED57-DOUT)
- LED59 pad 1: +5V -> Net-(LED59-DOUT)
- LED59 pad 2: Net-(LED59-DOU) -> +5V
- LED59 pad 4: Net-(LED58-DOU) -> Net-(LED58-DOUT)
- LED6 pad 1: +5V -> Net-(LED6-DOUT)
- LED6 pad 2: Net-(LED6-DOU) -> +5V
- LED6 pad 4: Net-(LED5-DOU) -> Net-(LED5-DOUT)
- LED60 pad 1: +5V -> Net-(LED60-DOUT)
- LED60 pad 2: Net-(LED60-DOU) -> +5V
- LED60 pad 4: Net-(LED59-DOU) -> Net-(LED59-DOUT)
- LED61 pad 1: +5V -> Net-(LED61-DOUT)
- LED61 pad 2: Net-(LED61-DOU) -> +5V
- LED61 pad 4: Net-(LED60-DOU) -> Net-(LED60-DOUT)
- LED62 pad 1: +5V -> Net-(LED62-DOUT)
- LED62 pad 2: Net-(LED62-DOU) -> +5V
- LED62 pad 4: Net-(LED61-DOU) -> Net-(LED61-DOUT)
- LED63 pad 1: +5V -> Net-(LED63-DOUT)
- LED63 pad 2: unconnected-(LED63-DOU-Pad2) -> +5V
- LED63 pad 4: Net-(LED62-DOU) -> Net-(LED62-DOUT)
- LED64 pad 1: +5V -> Net-(LED64-DOUT)
- LED64 pad 2: Net-(LED64-DOU) -> +5V
- LED64 pad 4: Net-(LED64-DIN) -> Net-(LED63-DOUT)
- LED65 pad 1: +5V -> Net-(LED65-DOUT)
- LED65 pad 2: unconnected-(LED65-DOU-Pad2) -> +5V
- LED65 pad 4: Net-(LED64-DOU) -> Net-(LED64-DOUT)
- LED7 pad 1: +5V -> Net-(LED7-DOUT)
- LED7 pad 2: Net-(LED7-DOU) -> +5V
- LED7 pad 4: Net-(LED6-DOU) -> Net-(LED6-DOUT)
- LED8 pad 1: +5V -> Net-(LED8-DOUT)
- LED8 pad 2: Net-(LED8-DOU) -> +5V
- LED8 pad 4: Net-(LED7-DOU) -> Net-(LED7-DOUT)
- LED9 pad 1: +5V -> Net-(LED10-DIN)
- LED9 pad 2: Net-(LED10-DIN) -> +5V
- LED9 pad 4: Net-(LED8-DOU) -> Net-(LED8-DOUT)
- U_CPU1 pad 23: LEDS_MILLENNIUM_LINE -> unconnected-(U_CPU1-IO15-Pad23)
- U_CPU1 pad 27: LEDS_CANADA_LINE -> unconnected-(U_CPU1-IO16-Pad27)
- U_CPU1 pad 28: LEDS_SEA_BUS_LINE -> unconnected-(U_CPU1-IO17-Pad28)
- U_CPU1 pad 30: SW_BRIGHTNESS -> unconnected-(U_CPU1-IO18-Pad30)
Routing:
- net +5V: track 0.00 -> 1671.2 mm

Commit message: Ground pins
Parts:
- removed C1, C123, C139, C141, C142, C2, C4: 1uF,25V,X5R, vancouver-skytrain-pcb.pretty:C_0402_1005Metric
- removed C103, C120, C137, C140, C3, C30, C5, C55, C79: 10uF,10V,X5R, vancouver-skytrain-pcb.pretty:C_0603_1608Metric
- removed D1: STATUS_LED, vancouver-skytrain-pcb.pretty:LED_0603_1608Metric
- removed J2_POWER_IN1: Conn_01x02, Connector_Phoenix_MC:PhoenixContact_MCV_1,5_2-G-3.81_1x02_P3.81mm_Vertical
- removed J3_PROGRAMING_PIN1: Conn_01x06, Connector_PinHeader_2.54mm:PinHeader_1x06_P2.54mm_Vertical
- removed Q1, Q2: PN2222A, Package_TO_SOT_SMD:SOT-416
- removed R1: 1k, vancouver-skytrain-pcb.pretty:C_0402_1005Metric
- removed R2, R3, R4: 10k, vancouver-skytrain-pcb.pretty:C_0402_1005Metric
- removed SW_BOOTLOAD1, SW_BRIGHTNESS1, SW_RESET1: Switch_SW_Push, Button_Switch_SMD:SW_Push_1P1T_NO_6x6mm_H9.5mm
- removed U1: 74AHC1G125, Package_TO_SOT_SMD:SOT-23-5
- removed U_CPU1: ESP32-WROOM-32E, RF_Module:ESP32-WROOM-32
- removed U_POWER1: LT1117-3.3, Package_TO_SOT_SMD:TO-263-3_TabPin2
- turned LED73 to -90 degrees
- turned LED81 to -90 degrees
Routing:
- net LEDS_CANADA_LINE_SOUTH_TO_NORTH: track 0.00 -> 260.5 mm, vias 0 -> 2
- net LEDS_MILLENNIUM_LINE_EAST_TO_WEST: track 0.00 -> 140.7 mm, vias 0 -> 2
- net GND: track 0.00 -> 118.8 mm, vias 0 -> 177
- net Net-(LED25-DOUT): track 0.00 -> 41.3 mm, vias 0 -> 2
- net Net-(LED15-DOUT): track 0.00 -> 39.6 mm, vias 0 -> 2
- net Net-(LED88-DOUT): track 0.00 -> 35.7 mm, vias 0 -> 2
- net Net-(LED54-DOUT): track 0.00 -> 30.8 mm, vias 0 -> 2
- net Net-(LED102-DOUT): track 0.00 -> 24.8 mm, vias 0 -> 2
- net Net-(LED117-DOUT): track 0.00 -> 23.1 mm
- net Net-(LED123-DOUT): track 0.00 -> 22.5 mm
- net Net-(LED4-DOUT): track 0.00 -> 22.3 mm
- net Net-(LED38-DOUT): track 0.00 -> 20.5 mm
- net Net-(LED53-DOUT): track 0.00 -> 19.6 mm
- net Net-(LED79-DOUT): track 0.00 -> 19.5 mm, vias 0 -> 2
- net Net-(LED109-DOUT): track 0.00 -> 18.8 mm
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- added copper zone on B.Cu, net GND
Other:
- board outline added: 300 x 191.8 mm

Commit message: Resolved a bunch of DRC errors
Parts:
- removed the G*** at (175.5, 124.9) (x3)
- added C1: 1uF,25V,X5R, vancouver-skytrain-pcb.pretty:C_0402_1005Metric, F.Cu at (239.2, 189.5)
- added C103: 1uF,25V,X5R, vancouver-skytrain-pcb.pretty:C_0402_1005Metric, F.Cu at (250.2, 172.2)
- added C120: 1uF,25V,X5R, vancouver-skytrain-pcb.pretty:C_0402_1005Metric, F.Cu at (250.2, 173.5)
- added C123: 1uF,25V,X5R, vancouver-skytrain-pcb.pretty:C_0402_1005Metric, F.Cu at (250.2, 176.0)
- added C2: 1uF,25V,X5R, vancouver-skytrain-pcb.pretty:C_0402_1005Metric, F.Cu at (285.5, 190.8)
- added C3: 10uF,10V,X5R, vancouver-skytrain-pcb.pretty:C_0603_1608Metric, F.Cu at (246.5, 185.0)
- added C30: 1uF,25V,X5R, vancouver-skytrain-pcb.pretty:C_0402_1005Metric, F.Cu at (250.2, 177.2)
- added C4: 1uF,25V,X5R, vancouver-skytrain-pcb.pretty:C_0402_1005Metric, F.Cu at (301.8, 174.6)
- added C5: 1uF,25V,X5R, vancouver-skytrain-pcb.pretty:C_0402_1005Metric, F.Cu at (117.0, 31.0)
- added C55: 1uF,25V,X5R, vancouver-skytrain-pcb.pretty:C_0402_1005Metric, F.Cu at (250.2, 174.8)
- added C79: 1uF,25V,X5R, vancouver-skytrain-pcb.pretty:C_0402_1005Metric, F.Cu at (250.2, 171.0)
- added D1: STATUS_LED, vancouver-skytrain-pcb.pretty:LED_0603_1608Metric, F.Cu at (280.5, 171.0)
- added G*** (x2): LOGO, LOGO, F.Cu at (161.9, 112.0)
- added H1: MountingHole, MountingHole:MountingHole_3.2mm_M3, F.Cu at (22.0, 22.0)
- added H2: MountingHole, MountingHole:MountingHole_3.2mm_M3, F.Cu at (302.0, 22.0)
- added H3: MountingHole, MountingHole:MountingHole_3.2mm_M3, F.Cu at (302.0, 190.0)
- added H4: MountingHole, MountingHole:MountingHole_3.2mm_M3, F.Cu at (22.0, 190.0)
- added J1: Conn_01x04, Connector_PinHeader_2.54mm:PinHeader_1x04_P2.54mm_Vertical, F.Cu at (308.8, 148.9)
- added J2_POWER_IN1: Conn_01x02, Connector_Phoenix_MC:PhoenixContact_MCV_1,5_2-G-3.81_1x02_P3.81mm_Vertical, F.Cu at (240.5, 194.0)
- added J3_PROGRAMING_PIN1: Conn_01x06, Connector_PinHeader_2.54mm:PinHeader_1x06_P2.54mm_Vertical, F.Cu at (308.8, 164.7)
- added LED127: WS2812B, vancouver-skytrain-pcb.pretty:XL-1010RGBC-WS2812B, F.Cu at (116.8, 32.8)
- added Q1: PN2222A, Package_TO_SOT_SMD:SOT-416, F.Cu at (299.0, 176.6)
- added Q2: PN2222A, Package_TO_SOT_SMD:SOT-416, F.Cu at (301.5, 176.6)
- added R1: 1k, vancouver-skytrain-pcb.pretty:C_0402_1005Metric, F.Cu at (278.0, 171.0)
- added R2: 0, Resistor_SMD:R_0402_1005Metric, F.Cu at (286.0, 176.0)
- added R3: 10k, vancouver-skytrain-pcb.pretty:C_0402_1005Metric, F.Cu at (298.5, 178.8)
- added R4: 10k, vancouver-skytrain-pcb.pretty:C_0402_1005Metric, F.Cu at (301.0, 178.8)
- added R5: 10k, vancouver-skytrain-pcb.pretty:C_0402_1005Metric, F.Cu at (298.8, 174.6)
- added SW_BOOTLOAD1: Switch_SW_Push, Button_Switch_SMD:SW_Push_1P1T_NO_6x6mm_H9.5mm, B.Cu at (272.0, 164.2)
- added SW_RESET1: Switch_SW_Push, Button_Switch_SMD:SW_Push_1P1T_NO_6x6mm_H9.5mm, B.Cu at (279.2, 164.2)
- added U1: 74AHC1G125, Package_TO_SOT_SMD:SOT-23-5, F.Cu at (299.2, 151.5)
- added U_CPU1: ESP32-WROOM-32E, RF_Module:ESP32-WROOM-32, F.Cu at (275.0, 183.0)
- added U_POWER1: LT1117-3.3, Package_TO_SOT_SMD:TO-263-3_TabPin2, F.Cu at (238.5, 176.4)
- moved C84 18.9 mm to (100.2, 141.0)
- moved LED44 18.7 mm to (245.7, 111.9)
- moved LED11 18.7 mm to (175.0, 124.2)
- moved LED12 18.7 mm to (167.5, 116.9)
- moved LED18 18.7 mm to (94.4, 59.1)
- moved C10 18.7 mm to (218.2, 138.2)
- moved C100 18.7 mm to (193.5, 90.9)
- moved C101 18.7 mm to (193.5, 93.9)
- moved C102 18.7 mm to (183.8, 90.8)
- moved C104 18.7 mm to (183.8, 94.0)
- moved C105 18.7 mm to (271.8, 60.5)
- moved C106 18.7 mm to (253.2, 94.5)
- moved C107 18.7 mm to (248.2, 94.5)
- moved C108 18.7 mm to (248.2, 91.0)
- moved C109 18.7 mm to (253.2, 91.0)
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Connections:
- LED126 pad 1: LED_OUT -> LEDS_SEA_BUS
Routing:
- net LED_OUT: track 0.00 -> 308.2 mm, vias 0 -> 2
- net +5V: track 1670.2 -> 1877.2 mm, vias 3 -> 12
- net LEDS_SEA_BUS: track 0.00 -> 165.2 mm, vias 0 -> 2
- net LEDS_CANADA_LINE_SOUTH_TO_NORTH: track 260.5 -> 348.3 mm
- net +3.3V: track 0.00 -> 84.7 mm, vias 0 -> 4
- net /TXD: track 0.00 -> 61.2 mm, vias 0 -> 2
- net /RXD: track 0.00 -> 60.5 mm, vias 0 -> 2
- net /RESET: track 0.00 -> 60.4 mm, vias 0 -> 2
- net /GPIO0: track 0.00 -> 59.7 mm, vias 0 -> 2
- net GND: track 118.8 -> 172.7 mm, vias 177 -> 195
- net LED_IN: track 0.00 -> 41.8 mm
- net LEDS_EXPO_LINE_EAST_TO_WEST: track 0.00 -> 40.0 mm, vias 0 -> 2
- net LEDS_MILLENNIUM_LINE_EAST_TO_WEST: track 140.7 -> 156.6 mm
- net /RTS: track 0.00 -> 11.8 mm, vias 0 -> 2
- net Net-(LED44-DOUT): track 16.9 -> 22.1 mm, vias 1 -> 2
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- added copper zone on F.Cu, net +3.3V
Other:
- board size 300 x 191.8 mm -> 300 x 188 mm
