File: hardware/vancouver-skytrain-pcb/vancouver-skytrain-pcb.kicad_pcb (KiCad board)
At the start: 2 copper layers, 300 x 188 mm, 286 parts, among them J1 Conn_01x04, J2_POWER_IN1 Conn_01x02, J3_PROGRAMING_PIN1 Conn_01x06, Q1 PN2222A, Q2 PN2222A, U1 74AHC1G125

Commit message: Clean up before sending to fab
Parts:
- removed the G*** at (161.9, 112.0) (x2)
- added G*** (x3): LOGO, LOGO, F.Cu at (161.9, 112.0)
- U_POWER1: value LT1117-3.3 -> UR133AG-33-AB3-C-R__3.3v; footprint Package_TO_SOT_SMD:TO-263-3_TabPin2 -> Package_TO_SOT_SMD:SOT-89-3
- moved SW_BOOTLOAD1 5.01 mm to (267.0, 164.2)
- moved U_POWER1 3.37 mm to (238.7, 179.8)
- moved SW_RESET1 2.98 mm to (282.2, 164.2)
- moved C2 0.24 mm to (285.5, 190.5)
Routing:
- net GND: track 172.7 -> 242.9 mm, vias 195 -> 197
- net +3.3V: track 84.7 -> 77.4 mm
- net /RESET: track 60.4 -> 53.7 mm
- net /GPIO0: track 59.7 -> 55.6 mm
- net Net-(LED117-DOUT): track 23.5 -> 21.8 mm
- net +5V: track 1877.2 -> 1878.5 mm, vias 12 -> 10
- net LED_IN: track 41.8 -> 41.2 mm
- net Net-(LED54-DOUT): track 31.0 -> 30.5 mm
- net Net-(LED104-DOUT): track 16.5 -> 17.0 mm, vias 0 -> 2
- net Net-(LED22-DOUT): track 18.1 -> 17.6 mm
- net Net-(LED68-DOUT): track 15.9 -> 15.4 mm
- net Net-(LED123-DOUT): track 22.6 -> 22.1 mm, vias 0 -> 2
- net Net-(LED116-DOUT): vias 0 -> 2
- added copper zone on F.Cu, net GND
- removed copper zone on F.Cu, net +3.3V
Other:
- board text added: "+3.3V"
- board text added: "+5V"
- board text added: "Author: Steven Smethurst @funvill Version: 2023-Sep-17 https://github.com/funvill/vancouver-skytrain-pcb Choo Choo"
- board text added: "GND"
- board text added: "GPIO 0"
- board text added: "LED_IN"
- board text added: "LED_OUT"
- board text added: "RESET"
- board text added: "RTS"
- board text added: "RXD"
- board text added: "TXD"

Commit message: Updated headers and update to kicad v8
Parts:
- added J2: Conn_01x02, Connector_PinHeader_2.54mm:PinHeader_1x02_P2.54mm_Vertical, F.Cu at (272.4, 163.2)
- added J3: Conn_01x02, Connector_PinHeader_2.54mm:PinHeader_1x02_P2.54mm_Vertical, F.Cu at (276.9, 163.3)
- added J4: Conn_01x09, Connector_PinHeader_2.54mm:PinHeader_1x08_P2.54mm_Vertical, F.Cu at (257.2, 167.9)
- J1: footprint Connector_PinHeader_2.54mm:PinHeader_1x04_P2.54mm_Vertical -> Connector_PinHeader_2.54mm:PinHeader_1x05_P2.54mm_Vertical
Connections:
- U_CPU1 pad 26: unconnected-(U_CPU1-IO4-Pad26) -> Pin26
- U_CPU1 pad 27: unconnected-(U_CPU1-IO16-Pad27) -> Pin27
- U_CPU1 pad 28: unconnected-(U_CPU1-IO17-Pad28) -> Pin28
- U_CPU1 pad 29: unconnected-(U_CPU1-IO5-Pad29) -> Pin29
- U_CPU1 pad 30: unconnected-(U_CPU1-IO18-Pad30) -> Pin30
- U_CPU1 pad 31: unconnected-(U_CPU1-IO19-Pad31) -> Pin31
- U_CPU1 pad 33: unconnected-(U_CPU1-IO21-Pad33) -> Pin33
- U_CPU1 pad 36: unconnected-(U_CPU1-IO22-Pad36) -> Pin36
Routing:
- net Pin26: track 0.00 -> 16.3 mm
- net Pin27: track 0.00 -> 11.9 mm
- net Pin28: track 0.00 -> 11.4 mm
- net Pin29: track 0.00 -> 10.9 mm
- net Pin36: track 0.00 -> 10.3 mm
- net Pin30: track 0.00 -> 10.3 mm
- net Pin33: track 0.00 -> 9.81 mm
- net Pin31: track 0.00 -> 9.81 mm
- net /RESET: track 53.7 -> 62.8 mm, vias 2 -> 3
- net /GPIO0: track 55.6 -> 64.4 mm
Other:
- board text added: "Author: Steven Smethurst @funvill Version: 2024-Mar-23 https://github.com/funvill/vancouver-skytrain-pcb Choo Choo"
- board text added: "JLCJLCJLCJLC"
- board text removed: "Author: Steven Smethurst @funvill Version: 2023-Sep-17 https://github.com/funvill/vancouver-skytrain-pcb Choo Choo"
