File: ai-v3/hardware/vancouver-skytrain-pcb.kicad_sch (KiCad schematic)
At the start: 85 parts, among them SW1 TS-1187A-B-A-B, SW2 TS-1187A-B-A-B, SW3 TS-1187A-B-A-B, SW4 TS-1187A-B-A-B, U1 XIAO-RP2040-DIP

Commit message: ai-v3: JLCPCB fabrication outputs
hardware/jlcpcb/: gerbers (9 layers, Protel extensions, mask-subtracted
silk) + Excellon drill and map zipped for the order page; BOM and CPL in
JLC's column format for SMT assembly, covering the 68 WS2812B LEDs
(C5349954) and 8 x 10uF 0402 (C52923) - switches are DNP, the XIAO is a
hand-soldered module. tools/make_jlcpcb.py derives the two JLC files
from kicad-cli's raw pos/BOM exports and builds the zip; README.md in
the folder has the upload map and the exact commands.

DRC at this state (KiCad 10.0.5): no unconnected items, no clearance /
edge / courtyard violations; remaining are the two no-net mounting holes
touching the water copper and two thin GND thermals (LED35, LED38).
Includes the user's +5V and GND zone routing fixes.

Co-Authored-By: Claude Fable 5.1 <noreply@anthropic.com>
Parts:
- added H1, H2, H3, H4: MountingHole, MountingHole:MountingHole_3.2mm_M3_DIN965_Pad_TopBottom, symbol Mechanical:MountingHole
- added ROW0: 10uF,10V,X5R, Capacitor_SMD:C_0402_1005Metric, symbol __sws_jlpcb:jlcpcb-1uF,25V,X5R
Connections:
- net +5V: now also ROW0.1
- net GND: now also ROW0.2
